File: starfield/starfield.kicad_sch (KiCad schematic)
At the start: 72 parts, among them J1 Screw_Terminal_01x02, J2 Screw_Terminal_01x02, J3 Conn_01x05_Socket, Q1 2N7002K, U3 LP5036

Commit message: code
Other:
- note added: "forgot a term calculating resistor values, expecting more like 4V"
- note added: "i know the pot says 50k on it but it really is measuring more like 44 or 45k also next time just use the 3 pin potentiometer to 3v3"
Changed lines of the file:
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@@
+		)
+	)
+	(text "i know the pot says 50k on it but it really is measuring more like 44 or 45k\nalso next time just use the 3 pin potentiometer to 3v3\n"
+		(exclude_from_sim no)
+		(at 56.388 29.972 0)
+		(effects
+			(font
+				(size 1.27 1.27)
+			)
 		)
 	)
@@
 		(effects
 			(font
+				(size 1.27 1.27)
+			)
+		)
+	)
+	(text "forgot a term calculating resistor values, expecting more like 4V"
+		(exclude_from_sim no)
+		(at 91.186 113.792 0)
+		(effects
+			(font
